Commit message: tidy up togo URDF

File: togo_description/urdf/togo.urdf.xacro (robot description, xacro)
@@ -1,5 +1,5 @@
 <?xml version="1.0"?>
-<robot xmlns:xacro="http://www.ros.org/wiki/xacro" name="a300-00058">
-<xacro:include filename="$(find togo_description)/urdf/togo_macro.xacro"/>
-<xacro:togo/>
+<robot xmlns:xacro="http://www.ros.org/wiki/xacro" name="togo">
+  <xacro:include filename="$(find togo_description)/urdf/togo_macro.xacro"/>
+  <xacro:togo/>
 </robot>

File: togo_description/urdf/togo_macro.xacro (robot description, xacro)
@@ -2,6 +2,9 @@
 <robot xmlns:xacro="http://www.ros.org/wiki/xacro">
   <xacro:macro name="togo">
+  <xacro:arg name="is_sim" default="false" />
   <!-- Common; let Clearpath own this -->
   <xacro:include filename="$(find clearpath_platform_description)/urdf/common.urdf.xacro"/>
+  <!-- if ignition or gazebo - need to use absolute paths instead of relative-->
+  <!-- <xacro:property name="force_abs_paths" value="$(arg is_sim)" scope="global" /> -->
   <!-- Platform -->
   <xacro:include filename="$(find togo_description)/urdf/a300/a300.urdf.xacro"/>
