Commit message: remove references to togo_gz package from description

File: togo_description/urdf/a300/a300.urdf.xacro (robot description, xacro)
@@ -3,5 +3,4 @@
   <xacro:arg name="namespace" default="" />
   <xacro:arg name="is_sim" default="false" />
-  <xacro:arg name="gazebo_controllers" default="$(find togo_gz)/config/gazebo_controllers.yaml"/>  <!-- TODO broken for Gazebo -->
   <xacro:arg name="use_platform_controllers" default="true"/>
   <!-- Global Variables -->

File: togo_description/urdf/a300/drivetrain/control/diff_fwd.urdf.xacro (robot description, xacro)
@@ -2,7 +2,4 @@
 <robot xmlns:xacro="http://ros.org/wiki/xacro" xmlns:gz="http://gazebosim.org/schema" name="generic_drivetrain_control_diff_fwd">
   <xacro:macro name="generic_drivetrain_control_diff_fwd" params="name hardware_plugin">
-    <!-- Gazebo Controller -->
-    <xacro:include filename="$(find togo_gz)/urdf/gazebo.urdf.xacro"/>
-    <!-- TODO not sure what to do with this or where it goes rn; under togo_gz -->
     <!-- ROS2 controls -->
     <ros2_control name="${name}_hardware" type="system">

File: togo_description/urdf/a300/drivetrain/control/diff_rwd.urdf.xacro (robot description, xacro)
@@ -2,7 +2,4 @@
 <robot xmlns:xacro="http://ros.org/wiki/xacro" xmlns:gz="http://gazebosim.org/schema" name="generic_drivetrain_control_diff_rwd">
   <xacro:macro name="generic_drivetrain_control_diff_rwd" params="name hardware_plugin">
-    <!-- Gazebo Controller -->
-    <xacro:include filename="$(find togo_gz)/urdf/gazebo.urdf.xacro"/>
-    <!-- TODO not sure what to do with this or where it goes rn; under togo_gz -->
     <!-- ROS2 controls -->
     <ros2_control name="${name}_hardware" type="system">

File: togo_description/urdf/a300/drivetrain/control/omni_4wd.urdf.xacro (robot description, xacro)
@@ -2,7 +2,4 @@
 <robot xmlns:xacro="http://ros.org/wiki/xacro" xmlns:gz="http://gazebosim.org/schema" name="generic_drivetrain_control_omni_4wd">
   <xacro:macro name="generic_drivetrain_control_omni_4wd" params="name hardware_plugin">
-    <!-- Gazebo Controller -->
-    <xacro:include filename="$(find togo_gz)/urdf/gazebo.urdf.xacro"/>
-    <!-- TODO not sure what to do with this or where it goes rn; under togo_gz -->
     <!-- ROS2 controls -->
     <ros2_control name="${name}_hardware" type="system">

File: togo_description/urdf/togo_macro.xacro (robot description, xacro)
@@ -5,6 +5,4 @@
   <!-- Common; let Clearpath own this -->
   <xacro:include filename="$(find clearpath_platform_description)/urdf/common.urdf.xacro"/>
-  <!-- if ignition or gazebo - need to use absolute paths instead of relative-->
-  <!-- <xacro:property name="force_abs_paths" value="$(arg is_sim)" scope="global" /> -->
   <!-- Platform -->
   <xacro:include filename="$(find togo_description)/urdf/a300/a300.urdf.xacro"/>

Commit message: use open source Clearpath description as much as possible

File: togo_description/urdf/a300/a300.urdf.xacro (robot description, xacro)
@@ -49,15 +49,15 @@
       <visual>
         <geometry>
-          <mesh filename="package://togo_description/meshes/a300/chassis.dae" />
+          <mesh filename="package://clearpath_platform_description/meshes/a300/chassis.dae" />
         </geometry>
       </visual>
       <visual>
         <geometry>
-          <mesh filename="package://togo_description/meshes/a300/livery.dae" />
+          <mesh filename="package://clearpath_platform_description/meshes/a300/livery.dae" />
         </geometry>
       </visual>
       <visual>
         <geometry>
-          <mesh filename="package://togo_description/meshes/a300/status_lights.dae" />
+          <mesh filename="package://clearpath_platform_description/meshes/a300/status_lights.dae" />
         </geometry>
       </visual>
@@ -65,5 +65,5 @@
         <material name="clearpath_yellow"/>
         <geometry>
-          <mesh filename="package://togo_description/meshes/a300/chassis_collision.stl" />
+          <mesh filename="package://clearpath_platform_description/meshes/a300/chassis_collision.stl" />
         </geometry>
       </collision>
@@ -116,9 +116,9 @@
     </joint>
     <!-- Suspension beams -->
-    <xacro:include filename="$(find togo_description)/urdf/a300/drivetrain/suspension_beam.urdf.xacro"/>
+    <xacro:include filename="$(find clearpath_platform_description)/urdf/a300/drivetrain/suspension_beam.urdf.xacro"/>
     <xacro:a300_suspension_beam side="left"/>
     <xacro:a300_suspension_beam side="right"/>
     <!-- Add wheels -->
-    <xacro:include filename="$(find togo_description)/urdf/a300/drivetrain/wheels.urdf.xacro"/>
+    <xacro:include filename="$(find clearpath_platform_description)/urdf/a300/drivetrain/wheels.urdf.xacro"/>
     <xacro:a300_drivetrain_wheels front_wheels="${front_wheels}" rear_wheels="${rear_wheels}"/>
     <!-- Add drivetrain -->

File: togo_description/urdf/togo_macro.xacro (robot description, xacro)
@@ -8,33 +8,33 @@
   <xacro:a300 control="diff_4wd" front_wheels="outdoor" rear_wheels="outdoor"/>
   <!-- Attachments -->
-  <xacro:include filename="$(find togo_description)/urdf/a300/attachments/bumper.urdf.xacro"/>
+  <xacro:include filename="$(find clearpath_platform_description)/urdf/a300/attachments/bumper.urdf.xacro"/>
   <xacro:bumper name="front_bumper" model="default" parent_link="front_bumper_mount" extension="0.0">
     <origin xyz="0.0 0.0 0.0" rpy="0.0 0.0 0.0"/>
   </xacro:bumper>
-  <xacro:include filename="$(find togo_description)/urdf/a300/attachments/bumper.urdf.xacro"/>
+  <xacro:include filename="$(find clearpath_platform_description)/urdf/a300/attachments/bumper.urdf.xacro"/>
   <xacro:bumper name="rear_bumper" model="default" parent_link="rear_bumper_mount" extension="0.0">
     <origin xyz="0.0 0.0 0.0" rpy="0.0 0.0 0.0"/>
   </xacro:bumper>
-  <xacro:include filename="$(find togo_description)/urdf/a300/attachments/amp_enclosure.urdf.xacro"/>
+  <xacro:include filename="$(find clearpath_platform_description)/urdf/a300/attachments/amp_enclosure.urdf.xacro"/>
   <xacro:amp_enclosure name="enclosure" model="amp_enclosure" parent_link="base_link">
     <origin xyz="0.0 0.0 0.0" rpy="0.0 0.0 0.0"/>
   </xacro:amp_enclosure>
-  <xacro:include filename="$(find togo_description)/urdf/a300/attachments/amp_sensor_arch.urdf.xacro"/>
+  <xacro:include filename="$(find clearpath_platform_description)/urdf/a300/attachments/amp_sensor_arch.urdf.xacro"/>
   <xacro:amp_sensor_arch name="sensor_arch" model="amp_sensor_arch" parent_link="enclosure_antenna_mount">
     <origin xyz="0.0 0.0 0.0" rpy="0.0 0.0 0.0"/>
   </xacro:amp_sensor_arch>
-  <xacro:include filename="$(find togo_description)/urdf/a300/attachments/spotlight.urdf.xacro"/>
+  <xacro:include filename="$(find clearpath_platform_description)/urdf/a300/attachments/spotlight.urdf.xacro"/>
   <xacro:spotlight name="driving_light_1" model="spotlight" parent_link="sensor_arch_front_left_corner_mount">
     <origin xyz="0.0 0.0 -0.08" rpy="0.0 0.5235987755982988 0.5235987755982988"/>
   </xacro:spotlight>
-  <xacro:include filename="$(find togo_description)/urdf/a300/attachments/spotlight.urdf.xacro"/>
+  <xacro:include filename="$(find clearpath_platform_description)/urdf/a300/attachments/spotlight.urdf.xacro"/>
   <xacro:spotlight name="driving_light_2" model="spotlight" parent_link="sensor_arch_front_right_corner_mount">
     <origin xyz="0.0 0.0 -0.08" rpy="0.0 0.5235987755982988 -0.5235987755982988"/>
   </xacro:spotlight>
-  <xacro:include filename="$(find togo_description)/urdf/a300/attachments/spotlight.urdf.xacro"/>
+  <xacro:include filename="$(find clearpath_platform_description)/urdf/a300/attachments/spotlight.urdf.xacro"/>
   <xacro:spotlight name="driving_light_3" model="spotlight" parent_link="sensor_arch_rear_left_corner_mount">
     <origin xyz="0.0 0.0 -0.08" rpy="0.0 0.5235987755982988 -0.5235987755982988"/>
   </xacro:spotlight>
-  <xacro:include filename="$(find togo_description)/urdf/a300/attachments/spotlight.urdf.xacro"/>
+  <xacro:include filename="$(find clearpath_platform_description)/urdf/a300/attachments/spotlight.urdf.xacro"/>
   <xacro:spotlight name="driving_light_4" model="spotlight" parent_link="sensor_arch_rear_right_corner_mount">
     <origin xyz="0.0 0.0 -0.08" rpy="0.0 0.5235987755982988 0.5235987755982988"/>
@@ -44,25 +44,25 @@
   <!-- Sensors -->
   <!-- lidar3d_0 -->
-  <xacro:include filename="$(find togo_description)/urdf/sensors/seyond_lidar.urdf.xacro"/>
+  <xacro:include filename="$(find clearpath_sensors_description)/urdf/seyond_lidar.urdf.xacro"/>
   <xacro:seyond_lidar name="lidar3d_0" parent_link="enclosure_front_lidar_mount" ang_res_h="0.01" ang_res_v="0.01" min_ang_h="-1.0471975511965976" max_ang_h="1.0471975511965976" min_ang_v="-0.6108652381980153" max_ang_v="0.6108652381980153" min_range="0.1" max_range="150.0" update_rate="20">
     <origin xyz="0.0 0.0 0.0" rpy="0.0 0.0 0.0"/>
   </xacro:seyond_lidar>
   <!-- camera_0 -->
-  <xacro:include filename="$(find togo_description)/urdf/sensors/luxonis_oakd.urdf.xacro"/>
+  <xacro:include filename="$(find clearpath_sensors_description)/urdf/luxonis_oakd.urdf.xacro"/>
   <xacro:luxonis_oakd name="camera_0" parent_link="sensor_arch_front_camera_mount" update_rate="30.0" model="pro">
     <origin xyz="0.0 0.0 0.0" rpy="0.0 0.0 0.0"/>
   </xacro:luxonis_oakd>
   <!-- camera_1 -->
-  <xacro:include filename="$(find togo_description)/urdf/sensors/luxonis_oakd.urdf.xacro"/>
+  <xacro:include filename="$(find clearpath_sensors_description)/urdf/luxonis_oakd.urdf.xacro"/>
   <xacro:luxonis_oakd name="camera_1" parent_link="sensor_arch_rear_camera_mount" update_rate="30.0" model="pro">
     <origin xyz="0.0 0.0 0.0" rpy="0.0 0.0 0.0"/>
   </xacro:luxonis_oakd>
   <!-- imu_0 -->
-  <xacro:include filename="$(find togo_description)/urdf/sensors/phidgets_spatial.urdf.xacro"/>
+  <xacro:include filename="$(find clearpath_sensors_description)/urdf/phidgets_spatial.urdf.xacro"/>
   <xacro:phidgets_spatial name="imu_0" parent_link="base_link">
     <origin xyz="0.059 0.0 0.161275" rpy="0.0 0.0 0.0"/>
   </xacro:phidgets_spatial>
   <!-- ins_0 -->
-  <xacro:include filename="$(find togo_description)/urdf/sensors/fixposition.urdf.xacro"/>
+  <xacro:include filename="$(find clearpath_sensors_description)/urdf/fixposition.urdf.xacro"/>
   <xacro:fixposition name="ins_0" parent_link="enclosure_ins_mount" num_antennas="2" gps_0_type="spherical" gps_0_xyz_x="0.0" gps_0_xyz_y="0.0" gps_0_xyz_z="0.0" gps_0_rpy_r="0.0" gps_0_rpy_p="0.0" gps_0_rpy_y="0.0" gps_0_parent="sensor_arch_right_antenna_mount" gps_1_type="spherical" gps_1_xyz_x="0.0" gps_1_xyz_y="0.0" gps_1_xyz_z="0.0" gps_1_rpy_r="0.0" gps_1_rpy_p="0.0" gps_1_rpy_y="0.0" gps_1_parent="sensor_arch_left_antenna_mount">
     <origin xyz="0.0 0.0 0.0" rpy="0.0 0.0 0.0"/>
